File: BitDisplay/BitDisplay.sch (KiCad schematic (older format))
At the start: 13 parts, among them J0 Power Hdr, J1 Bit Hdr, J2 Analog Hdr, SW0 Aux, SW1 Disp Mode, SW2 Input Mode

Commit message: PowerSupplyV1
Parts:
- A1: symbol 0_Usefull_Stuff:I2C_GPIO_8x -> 0-Components:I2C_GPIO_8x
Changed lines of the file:
@@
 	5650 2650 5650 2550
 $Comp
-L 0_Usefull_Stuff:I2C_GPIO_8x A1
+L 0-Components:I2C_GPIO_8x A1
 U 1 1 605B0983
 P 5700 3000
